File: Resources/LED_resistor.sch (EAGLE design)
At the start: 2 parts

Commit message: Added junctions and multi-line texts
Other:
- note added: "Simple text"
Changed lines of the file:
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@@
 <sheet>
 <plain>
+<text x="30.48" y="22.86" size="1.778" layer="97" rot="R90">Simple
+text</text>
 </plain>
 <instances>
@@
 <pinref part="R1" gate="G$1" pin="1"/>
 <pinref part="GND1" gate="1" pin="GND"/>
-<wire x1="10.16" y1="10.16" x2="10.16" y2="5.08" width="0.1524" layer="91"/>
-</segment>
-<segment>
-<wire x1="22.86" y1="5.08" x2="22.86" y2="12.7" width="0.1524" layer="91"/>
+<wire x1="10.16" y1="10.16" x2="10.16" y2="7.62" width="0.1524" layer="91"/>
+<wire x1="10.16" y1="7.62" x2="10.16" y2="5.08" width="0.1524" layer="91"/>
+<wire x1="22.86" y1="5.08" x2="22.86" y2="7.62" width="0.1524" layer="91"/>
+<wire x1="22.86" y1="7.62" x2="22.86" y2="12.7" width="0.1524" layer="91"/>
 <wire x1="22.86" y1="12.7" x2="30.48" y2="12.7" width="0.1524" layer="91"/>
 <label x="25.4" y="5.08" size="1.778" layer="95" rot="R90"/>
+<wire x1="10.16" y1="7.62" x2="22.86" y2="7.62" width="0.1524" layer="91"/>
+<junction x="10.16" y="7.62"/>
+<junction x="22.86" y="7.62"/>
 </segment>
 <segment>
@@
 </schematic>
 </drawing>
+<compatibility>
+<note version="6.3" minversion="6.2.2" severity="warning">
+Since Version 6.2.2 text objects can contain more than one line,
+which will not be processed correctly with this version.
+</note>
+</compatibility>
 </eagle>
